Commit message: Added robot resting position in planning
We can now manually set resting position in moveit

File: ros2_ws/src/ros2_kortex/kortex_description/robots/final_gen3_robotiq_2f_85.urdf (robot description, URDF)
Before this commit: robot gen3_robotiq_2f_85, 46 links, 45 joints
Links:
- added link box_link, mass 1.0; collision box size=0.5 0.5 0.5; visual box size=0.5 0.5 0.5
Joints:
- added joint box_joint: type fixed, parent world, child box_link, origin xyz=0 0 1.18 rpy=0 0 0

Commit message: Update final_gen3_robotiq_2f_85.urdf

File: ros2_ws/src/ros2_kortex/kortex_description/robots/final_gen3_robotiq_2f_85.urdf (robot description, URDF)
Before this commit: robot gen3_robotiq_2f_85, 47 links, 46 joints
Links:
- removed link box_link
- added link bound_left_link, mass 1.0; collision box size=2 0.05 0.05; visual box size=2 0.05 0.05
- added link bound_right_link, mass 1.0; collision box size=2 0.05 0.05; visual box size=2 0.05 0.05
- added link bound_top_link, mass 1.0; collision box size=2 0.05 0.05; visual box size=2 0.05 0.05
Joints:
- removed joint box_joint
- added joint bound_left_joint: type fixed, parent world, child bound_left_link, origin xyz=0.75 0 1.8 rpy=0 0 1.5708
- added joint bound_right_joint: type fixed, parent world, child bound_right_link, origin xyz=-0.73 0 1.8 rpy=0 0 1.5708
- added joint bound_top_joint: type fixed, parent world, child bound_top_link, origin xyz=0 0 1.8 rpy=0 0 0

Commit message: manually added obstacles and resting position

File: ros2_ws/src/ros2_kortex/kortex_description/robots/final_gen3_robotiq_2f_85.urdf (robot description, URDF)
Before this commit: robot gen3_robotiq_2f_85, 49 links, 48 joints
Links:
- added link bound_left_top_link, mass 1.0; collision box size=2 0.05 0.05; visual box size=2 0.05 0.05
- added link bound_right_top_link, mass 1.0; collision box size=2 0.05 0.05; visual box size=2 0.05 0.05
Joints:
- added joint bound_left_top_joint: type fixed, parent world, child bound_left_top_link, origin xyz=0.75 0 2.03 rpy=0 0 1.5708
- added joint bound_right_top_joint: type fixed, parent world, child bound_right_top_link, origin xyz=-0.7 0 2.03 rpy=0 0 1.5708
- joint bound_right_joint: origin xyz=-0.73 0 1.8 rpy=0 0 1.5708 -> xyz=-0.7 0 1.8 rpy=0 0 1.5708

Commit message: all bars added for collision avoidance

File: ros2_ws/src/ros2_kortex/kortex_description/robots/final_gen3_robotiq_2f_85.urdf (robot description, URDF)
Before this commit: robot gen3_robotiq_2f_85, 51 links, 50 joints
Links:
- added link bound_stand_1_link, mass 1.0; collision box size=2 0.1 0.1; visual box size=2 0.1 0.1
- added link bound_stand_2_link, mass 1.0; collision box size=2 0.1 0.1; visual box size=2 0.1 0.1
- added link bound_stand_3_link, mass 1.0; collision box size=2 0.1 0.1; visual box size=2 0.1 0.1
- added link bound_stand_4_link, mass 1.0; collision box size=2 0.1 0.1; visual box size=2 0.1 0.1
Joints:
- added joint bound_stand_1_joint: type fixed, parent world, child bound_stand_1_link, origin xyz=0.75 -0.55 1.1 rpy=0 1.5708 0
- added joint bound_stand_2_joint: type fixed, parent world, child bound_stand_2_link, origin xyz=-0.7 -0.55 1.1 rpy=0 1.5708 0
- added joint bound_stand_3_joint: type fixed, parent world, child bound_stand_3_link, origin xyz=-0.7 0.55 1.1 rpy=0 1.5708 0
- added joint bound_stand_4_joint: type fixed, parent world, child bound_stand_4_link, origin xyz=0.75 0.55 1.1 rpy=0 1.5708 0

Commit message: clean up ton of stuff, move control stack into ros workspace, dynamic stl files

File: ros2_ws/src/ros2_kortex/kortex_description/robots/final_gen3_robotiq_2f_85.urdf (robot description, URDF)
Before this commit: robot gen3_robotiq_2f_85, 55 links, 54 joints
Links:
- link left_base_link: geometry collision mesh filename=package://kortex_description/arms/gen3/7dof/meshes/base_lin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; visual mesh filename=package://kortex_description/arms/gen3/7dof/meshes/base_lin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
- link left_bracelet_link: geometry collision mesh filename=package://kortex_description/arms/gen3/7dof/meshes/bracelet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; visual mesh filename=package://kortex_description/arms/gen3/7dof/meshes/bracelet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
- link left_forearm_link: geometry collision mesh filename=package://kortex_description/arms/gen3/7dof/meshes/forearm_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; visual mesh filename=package://kortex_description/arms/gen3/7dof/meshes/forearm_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
- link left_half_arm_1_link: geometry collision mesh filename=package://kortex_description/arms/gen3/7dof/meshes/half_arm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; visual mesh filename=package://kortex_description/arms/gen3/7dof/meshes/half_arm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
- link left_half_arm_2_link: geometry collision mesh filename=package://kortex_description/arms/gen3/7dof/meshes/half_arm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; visual mesh filename=package://kortex_description/arms/gen3/7dof/meshes/half_arm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
- link left_robotiq_85_base_link: geometry collision mesh filename=package://robotiq_description/meshes/collision/2f_85/roboti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; visual mesh filename=package://robotiq_description/meshes/visual/2f_85/robotiq_b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
- link left_robotiq_85_left_finger_link: geometry collision mesh filename=package://robotiq_description/meshes/collision/2f_85/left_f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; visual mesh filename=package://robotiq_description/meshes/visual/2f_85/left_fing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
- link left_robotiq_85_left_finger_tip_link: geometry collision mesh filename=package://robotiq_description/meshes/collision/2f_85/left_f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; visual mesh filename=package://robotiq_description/meshes/visual/2f_85/left_fing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
- link left_robotiq_85_left_inner_knuckle_link: geometry collision mesh filename=package://robotiq_description/meshes/collision/2f_85/left_i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; visual mesh filename=package://robotiq_description/meshes/visual/2f_85/left_inne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
- link left_robotiq_85_left_knuckle_link: geometry collision mesh filename=package://robotiq_description/meshes/collision/2f_85/left_k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; visual mesh filename=package://robotiq_description/meshes/visual/2f_85/left_knuc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
- link left_robotiq_85_right_finger_link: geometry collision mesh filename=package://robotiq_description/meshes/collision/2f_85/right_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; visual mesh filename=package://robotiq_description/meshes/visual/2f_85/right_fin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
- link left_robotiq_85_right_finger_tip_link: geometry collision mesh filename=package://robotiq_description/meshes/collision/2f_85/right_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; visual mesh filename=package://robotiq_description/meshes/visual/2f_85/right_fin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
- link left_robotiq_85_right_inner_knuckle_link: geometry collision mesh filename=package://robotiq_description/meshes/collision/2f_85/right_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; visual mesh filename=package://robotiq_description/meshes/visual/2f_85/right_inn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
- link left_robotiq_85_right_knuckle_link: geometry collision mesh filename=package://robotiq_description/meshes/collision/2f_85/right_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; visual mesh filename=package://robotiq_description/meshes/visual/2f_85/right_knu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
- link left_shoulder_link: geometry collision mesh filename=package://kortex_description/arms/gen3/7dof/meshes/shoulder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; visual mesh filename=package://kortex_description/arms/gen3/7dof/meshes/shoulder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
- link left_spherical_wrist_1_link: geometry collision mesh filename=package://kortex_description/arms/gen3/7dof/meshes/spherica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; visual mesh filename=package://kortex_description/arms/gen3/7dof/meshes/spherica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
- link left_spherical_wrist_2_link: geometry collision mesh filename=package://kortex_description/arms/gen3/7dof/meshes/spherica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; visual mesh filename=package://kortex_description/arms/gen3/7dof/meshes/spherica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
- link right_base_link: geometry collision mesh filename=package://kortex_description/arms/gen3/7dof/meshes/base_lin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; visual mesh filename=package://kortex_description/arms/gen3/7dof/meshes/base_lin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
- link right_bracelet_link: geometry collision mesh filename=package://kortex_description/arms/gen3/7dof/meshes/bracelet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; visual mesh filename=package://kortex_description/arms/gen3/7dof/meshes/bracelet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
- link right_forearm_link: geometry collision mesh filename=package://kortex_description/arms/gen3/7dof/meshes/forearm_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; visual mesh filename=package://kortex_description/arms/gen3/7dof/meshes/forearm_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
- link right_half_arm_1_link: geometry collision mesh filename=package://kortex_description/arms/gen3/7dof/meshes/half_arm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; visual mesh filename=package://kortex_description/arms/gen3/7dof/meshes/half_arm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
- link right_half_arm_2_link: geometry collision mesh filename=package://kortex_description/arms/gen3/7dof/meshes/half_arm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; visual mesh filename=package://kortex_description/arms/gen3/7dof/meshes/half_arm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
- link right_robotiq_85_base_link: geometry collision mesh filename=package://robotiq_description/meshes/collision/2f_85/roboti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; visual mesh filename=package://robotiq_description/meshes/visual/2f_85/robotiq_b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
- link right_robotiq_85_left_finger_link: geometry collision mesh filename=package://robotiq_description/meshes/collision/2f_85/left_f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; visual mesh filename=package://robotiq_description/meshes/visual/2f_85/left_fing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
- link right_robotiq_85_left_finger_tip_link: geometry collision mesh filename=package://robotiq_description/meshes/collision/2f_85/left_f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; visual mesh filename=package://robotiq_description/meshes/visual/2f_85/left_fing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
- link right_robotiq_85_left_inner_knuckle_link: geometry collision mesh filename=package://robotiq_description/meshes/collision/2f_85/left_i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; visual mesh filename=package://robotiq_description/meshes/visual/2f_85/left_inne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
- link right_robotiq_85_left_knuckle_link: geometry collision mesh filename=package://robotiq_description/meshes/collision/2f_85/left_k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; visual mesh filename=package://robotiq_description/meshes/visual/2f_85/left_knuc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
- link right_robotiq_85_right_finger_link: geometry collision mesh filename=package://robotiq_description/meshes/collision/2f_85/right_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; visual mesh filename=package://robotiq_description/meshes/visual/2f_85/right_fin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
- link right_robotiq_85_right_finger_tip_link: geometry collision mesh filename=package://robotiq_description/meshes/collision/2f_85/right_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; visual mesh filename=package://robotiq_description/meshes/visual/2f_85/right_fin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
- link right_robotiq_85_right_inner_knuckle_link: geometry collision mesh filename=package://robotiq_description/meshes/collision/2f_85/right_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; visual mesh filename=package://robotiq_description/meshes/visual/2f_85/right_inn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
- link right_robotiq_85_right_knuckle_link: geometry collision mesh filename=package://robotiq_description/meshes/collision/2f_85/right_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; visual mesh filename=package://robotiq_description/meshes/visual/2f_85/right_knu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
- link right_shoulder_link: geometry collision mesh filename=package://kortex_description/arms/gen3/7dof/meshes/shoulder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; visual mesh filename=package://kortex_description/arms/gen3/7dof/meshes/shoulder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
- link right_spherical_wrist_1_link: geometry collision mesh filename=package://kortex_description/arms/gen3/7dof/meshes/spherica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; visual mesh filename=package://kortex_description/arms/gen3/7dof/meshes/spherica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
- link right_spherical_wrist_2_link: geometry collision mesh filename=package://kortex_description/arms/gen3/7dof/meshes/spherica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; visual mesh filename=package://kortex_description/arms/gen3/7dof/meshes/spherica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
- link vention_table_link: geometry collision mesh filename=package://control/kinova_gen3_mujoco/assets/VentionAssembly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 scale=0.001 0.001 0.001; visual mesh filename=package://control/kinova_gen3_mujoco/assets/VentionAssembly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 scale=0.001 0.001 0.001

Commit message: git ignore

File: ros2_ws/src/ros2_kortex/kortex_description/robots/final_gen3_robotiq_2f_85.urdf (robot description, URDF)
Before this commit: robot gen3_robotiq_2f_85, 47 links, 46 joints
Links:
- removed link left_gripper_planning_point
- removed link right_gripper_planning_point
Joints:
- removed joint left_gripper_planning_joint
- removed joint right_gripper_planning_joint
- joint bin_joint: type fixed -> floating

Commit message: fixed errors with moveit

File: ros2_ws/src/ros2_kortex/kortex_description/robots/final_gen3_robotiq_2f_85.urdf (robot description, URDF)
Before this commit: robot gen3_robotiq_2f_85, 45 links, 44 joints
Links:
- link world: geometry collision sphere radius=0.01; visual sphere radius=0.01
