Commit message: get moveit to execute trajectory with fake hardware! and get rid of redundant manip folder

File: ros2_ws/src/ros2_kortex/kortex_description/grippers/robotiq_2f_85/urdf/robotiq_2f_85_macro.xacro (robot description, xacro)
@@ -20,5 +20,5 @@
     </xacro:if>
     <xacro:robotiq_gripper
-        name="RobotiqGripperHardwareInterface"
+        name="${prefix}RobotiqGripperHardwareInterface"
         prefix="${prefix}"
         parent="${parent}"

File: ros2_ws/src/two_arm_moveit2_config/urdf/final_gen3_robotiq_2f_85.urdf (robot description, URDF)
Before this commit: robot gen3_robotiq_2f_85, 45 links, 44 joints
Joints:
- joint bin_joint: type floating -> fixed
