Commit message: mujoco integration

File: ros2_ws/src/ros2_kortex/kortex_description/arms/gen3/7dof/urdf/gen3_macro.xacro (robot description, xacro)
@@ -23,4 +23,5 @@
     use_fake_hardware:=false
     fake_sensor_commands:=false
+    sim_mujoco:=false
     sim_gazebo:=false
     sim_ignition:=false
@@ -37,4 +38,5 @@
       use_fake_hardware="${use_fake_hardware}"
       fake_sensor_commands="${fake_sensor_commands}"
+      sim_mujoco="${sim_mujoco}"
       sim_gazebo="${sim_gazebo}"
       sim_ignition="${sim_ignition}"

File: ros2_ws/src/ros2_kortex/kortex_description/arms/gen3/7dof/urdf/kortex.ros2_control.xacro (robot description, xacro)
@@ -6,4 +6,5 @@
     use_fake_hardware:=false
     fake_sensor_commands:=false
+    sim_mujoco:=false
     sim_gazebo:=false
     sim_ignition:=false
@@ -27,4 +28,7 @@
     <ros2_control name="${name}" type="system">
       <hardware>
+        <xacro:if value="${sim_mujoco}">
+          <plugin>mujoco_ros2_control/MujocoSystem</plugin>
+        </xacro:if>
         <xacro:if value="${sim_gazebo}">
           <plugin>gazebo_ros2_control/GazeboSystem</plugin>
@@ -43,5 +47,5 @@
           <param name="state_following_offset">0.0</param>
         </xacro:if>
-        <xacro:unless value="${use_fake_hardware or sim_gazebo or sim_ignition or sim_isaac}">
+        <xacro:unless value="${use_fake_hardware or sim_gazebo or sim_ignition or sim_isaac or sim_mujoco}">
           <plugin>kortex_driver/KortexMultiInterfaceHardware</plugin>
           <param name="robot_ip">${robot_ip}</param>
@@ -60,81 +64,151 @@
       </hardware>
       <joint name="${prefix}joint_1">
-        <command_interface name="position">
-          <param name="min">{-2*pi}</param>
-          <param name="max">{2*pi}</param>
-        </command_interface>
+        <!-- <xacro:if value="${sim_mujoco}">
+          <param name="position_kp">3000</param>
+          <param name="position_ki">1</param>
+          <param name="position_kd">100</param>
+          <param name="position_i_max">10000</param>
+          <command_interface name="position_pid"/>
+        </xacro:if> -->
+        <xacro:unless value="${sim_mujoco}">
+          <command_interface name="position">
+            <param name="min">{-2*pi}</param>
+            <param name="max">{2*pi}</param>
+          </command_interface>
+        </xacro:unless>
+        <command_interface name="position"/>
         <state_interface name="position">
           <param name="initial_value">${initial_positions['joint_1']}</param>
         </state_interface>
         <state_interface name="velocity"/>
-        <state_interface name="effort"/>
+        <!-- <state_interface name="effort"/> -->
       </joint>
       <joint name="${prefix}joint_2">
-        <command_interface name="position">
-          <param name="min">-2.41</param>
-          <param name="max">2.41</param>
-        </command_interface>
+        <!-- <xacro:if value="${sim_mujoco}">
+          <param name="position_kp">3000</param>
+          <param name="position_ki">1</param>
+          <param name="position_kd">100</param>
+          <param name="position_i_max">10000</param>
+          <command_interface name="position_pid"/>
+        </xacro:if> -->
+        <xacro:unless value="${sim_mujoco}">
+          <command_interface name="position">
+            <param name="min">-2.41</param>
+            <param name="max">2.41</param>
+          </command_interface>
+        </xacro:unless>
+        <command_interface name="position"/>
         <state_interface name="position">
           <param name="initial_value">${initial_positions['joint_2']}</param>
         </state_interface>
         <state_interface name="velocity"/>
-        <state_interface name="effort"/>
+        <!-- <state_interface name="effort"/> -->
       </joint>
       <joint name="${prefix}joint_3">
-        <command_interface name="position">
-          <param name="min">{-2*pi}</param>
-          <param name="max">{2*pi}</param>
-        </command_interface>
+        <!-- <xacro:if value="${sim_mujoco}">
+          <param name="position_kp">3000</param>
+          <param name="position_ki">1</param>
+          <param name="position_kd">100</param>
+          <param name="position_i_max">10000</param>
+          <command_interface name="position_pid"/>
+        </xacro:if> -->
+        <xacro:unless value="${sim_mujoco}">
+          <command_interface name="position">
+            <param name="min">{-2*pi}</param>
+            <param name="max">{2*pi}</param>
+          </command_interface>
+        </xacro:unless>
+        <command_interface name="position"/>
         <state_interface name="position">
           <param name="initial_value">${initial_positions['joint_3']}</param>
         </state_interface>
         <state_interface name="velocity"/>
-        <state_interface name="effort"/>
+        <!-- <state_interface name="effort"/> -->
       </joint>
       <joint name="${prefix}joint_4">
-        <command_interface name="position">
-          <param name="min">-2.66</param>
-          <param name="max">2.66</param>
-        </command_interface>
+        <!-- <xacro:if value="${sim_mujoco}">
+          <param name="position_kp">3000</param>
+          <param name="position_ki">1</param>
+          <param name="position_kd">100</param>
+          <param name="position_i_max">10000</param>
+          <command_interface name="position_pid"/>
+        </xacro:if> -->
+        <xacro:unless value="${sim_mujoco}">
+          <command_interface name="position">
+            <param name="min">-2.66</param>
+            <param name="max">2.66</param>
+          </command_interface>
+        </xacro:unless>
+        <command_interface name="position"/>
         <state_interface name="position">
           <param name="initial_value">${initial_positions['joint_4']}</param>
         </state_interface>
         <state_interface name="velocity"/>
-        <state_interface name="effort"/>
+        <!-- <state_interface name="effort"/> -->
       </joint>
       <joint name="${prefix}joint_5">
-        <command_interface name="position">
-          <param name="min">{-2*pi}</param>
-          <param name="max">{2*pi}</param>
-        </command_interface>
+        <!-- <xacro:if value="${sim_mujoco}">
+          <param name="position_kp">3000</param>
+          <param name="position_ki">1</param>
+          <param name="position_kd">100</param>
+          <param name="position_i_max">10000</param>
+          <command_interface name="position_pid"/>
+        </xacro:if> -->
+        <xacro:unless value="${sim_mujoco}">
+          <command_interface name="position">
+            <param name="min">{-2*pi}</param>
+            <param name="max">{2*pi}</param>
+          </command_interface>
+        </xacro:unless>
+        <command_interface name="position"/>
         <state_interface name="position">
           <param name="initial_value">${initial_positions['joint_5']}</param>
         </state_interface>
         <state_interface name="velocity"/>
-        <state_interface name="effort"/>
+        <!-- <state_interface name="effort"/> -->
       </joint>
       <joint name="${prefix}joint_6">
-        <command_interface name="position">
-          <param name="min">-2.23</param>
-          <param name="max">2.23</param>
-        </command_interface>
+        <!-- <xacro:if value="${sim_mujoco}">
+          <param name="position_kp">3000</param>
+          <param name="position_ki">1</param>
+          <param name="position_kd">100</param>
+          <param name="position_i_max">10000</param>
+          <command_interface name="position_pid"/>
+        </xacro:if> -->
+        <xacro:unless value="${sim_mujoco}">
+          <command_interface name="position">
+            <param name="min">-2.23</param>
+            <param name="max">2.23</param>
+          </command_interface>
+        </xacro:unless>
+        <command_interface name="position"/>
         <state_interface name="position">
           <param name="initial_value">${initial_positions['joint_6']}</param>
         </state_interface>
         <state_interface name="velocity"/>
-        <state_interface name="effort"/>
+        <!-- <state_interface name="effort"/> -->
       </joint>
       <joint name="${prefix}joint_7">
-        <command_interface name="position">
-          <param name="min">{-2*pi}</param>
-          <param name="max">{2*pi}</param>
-        </command_interface>
+        <!-- <xacro:if value="${sim_mujoco}">
+          <param name="position_kp">3000</param>
+          <param name="position_ki">1</param>
+          <param name="position_kd">100</param>
+          <param name="position_i_max">10000</param>
+          <command_interface name="position_pid"/>
+        </xacro:if> -->
+        <xacro:unless value="${sim_mujoco}">
+          <command_interface name="position">
+            <param name="min">{-2*pi}</param>
+            <param name="max">{2*pi}</param>
+          </command_interface>
+        </xacro:unless>
+        <command_interface name="position"/>
         <state_interface name="position">
           <param name="initial_value">${initial_positions['joint_7']}</param>
         </state_interface>
         <state_interface name="velocity"/>
-        <state_interface name="effort"/>
-      </joint>
-      <xacro:unless value="${use_fake_hardware or sim_gazebo or sim_ignition or sim_isaac}">
+        <!-- <state_interface name="effort"/> -->
+      </joint>
+      <xacro:unless value="${use_fake_hardware or sim_gazebo or sim_ignition or sim_isaac or sim_mujoco}">
         <xacro:if value="${use_internal_bus_gripper_comm}">
           <joint name="${prefix}${gripper_joint_name}">

File: ros2_ws/src/ros2_kortex/kortex_description/grippers/robotiq_2f_85/urdf/robotiq_2f_85_macro.xacro (robot description, xacro)
@@ -6,4 +6,5 @@
     use_fake_hardware:=false
     fake_sensor_commands:=false
+    sim_mujoco:=false
     sim_ignition:=false
     sim_isaac:=false
@@ -16,5 +17,5 @@
     <!-- Hardware talks directly to the gripper so we don't need ros2_control unless we are simulating -->
     <xacro:property name="include_ros2_control" value="false"/>
-    <xacro:if value="${sim_ignition or sim_isaac or use_fake_hardware or not use_internal_bus_gripper_comm}">
+    <xacro:if value="${sim_mujoco or sim_ignition or sim_isaac or use_fake_hardware or not use_internal_bus_gripper_comm}">
       <xacro:property name="include_ros2_control" value="true"/>
     </xacro:if>
@@ -27,4 +28,5 @@
         use_fake_hardware="${use_fake_hardware}"
         fake_sensor_commands="${fake_sensor_commands}"
+        sim_mujoco="${sim_mujoco}"
         sim_ignition="${sim_ignition}"
         sim_isaac="${sim_isaac}"

File: ros2_ws/src/ros2_kortex/kortex_description/robots/gen3.xacro (robot description, xacro)
@@ -16,4 +16,5 @@
     <xacro:arg name="gripper_max_velocity" default="100.0" />
     <xacro:arg name="gripper_max_force" default="100.0" />
+    <xacro:arg name="sim_mujoco" default="false" />
     <xacro:arg name="sim_gazebo" default="false" />
     <xacro:arg name="sim_ignition" default="false" />
@@ -50,4 +51,5 @@
         use_fake_hardware="$(arg use_fake_hardware)"
         fake_sensor_commands="$(arg fake_sensor_commands)"
+        sim_mujoco="$(arg sim_mujoco)"
         sim_gazebo="$(arg sim_gazebo)"
         sim_ignition="$(arg sim_ignition)"

File: ros2_ws/src/ros2_kortex/kortex_description/robots/kortex_robot.xacro (robot description, xacro)
@@ -21,4 +21,5 @@
     fake_sensor_commands:=false
     sim:=false
+    sim_mujoco:=false
     sim_gazebo:=false
     sim_ignition:=false
@@ -50,4 +51,5 @@
       use_fake_hardware="${use_fake_hardware}"
       fake_sensor_commands="${fake_sensor_commands}"
+      sim_mujoco="${sim_mujoco}"
       sim_gazebo="${sim_gazebo}"
       sim_ignition="${sim_ignition}"
@@ -82,4 +84,5 @@
         use_fake_hardware="${use_fake_hardware}"
         fake_sensor_commands="${fake_sensor_commands}"
+        sim_mujoco="${sim_mujoco}"
         sim_ignition="${sim_ignition}"
         sim_isaac="${sim_isaac}"

File: ros2_ws/src/ros2_robotiq_gripper/robotiq_description/urdf/2f_85.ros2_control.xacro (robot description, xacro)
@@ -4,4 +4,5 @@
         name
         prefix
+        sim_mujoco:=false
         sim_ignition:=false
         sim_isaac:=false
@@ -22,4 +23,7 @@
                     <param name="trigger_joint_command_threshold">0.02</param>
                 </xacro:if>
+                <xacro:if value="${sim_mujoco}">
+                    <plugin>mujoco_ros2_control/MujocoSystem</plugin>
+                </xacro:if>
                 <xacro:if value="${sim_ignition}">
                     <plugin>ign_ros2_control/IgnitionSystem</plugin>
@@ -30,5 +34,5 @@
                     <param name="state_following_offset">0.0</param>
                 </xacro:if>
-                <xacro:unless value="${use_fake_hardware or sim_ignition or sim_isaac}">
+                <xacro:unless value="${use_fake_hardware or sim_ignition or sim_isaac or sim_mujoco}">
                     <plugin>robotiq_driver/RobotiqGripperHardwareInterface</plugin>
                     <param name="gripper_closed_position">0.7929</param>
@@ -48,9 +52,9 @@
             </joint>
             <!-- When simulating we need to include the rest of the gripper joints -->
-            <xacro:if value="${use_fake_hardware or sim_isaac or sim_ignition}">
+            <xacro:if value="${use_fake_hardware or sim_isaac or sim_ignition or sim_mujoco}">
                 <joint name="${prefix}robotiq_85_right_knuckle_joint">
                     <param name="mimic">${prefix}robotiq_85_left_knuckle_joint</param>
                     <param name="multiplier">-1</param>
-                    <xacro:unless value="${sim_ignition}">
+                    <xacro:unless value="${sim_ignition or sim_mujoco}">
                         <command_interface name="position"/>
                         <state_interface name="position"/>
@@ -61,5 +65,5 @@
                     <param name="mimic">${prefix}robotiq_85_left_knuckle_joint</param>
                     <param name="multiplier">1</param>
-                    <xacro:unless value="${sim_ignition}">
+                    <xacro:unless value="${sim_ignition or sim_mujoco}">
                         <command_interface name="position"/>
                         <state_interface name="position"/>
@@ -70,5 +74,5 @@
                     <param name="mimic">${prefix}robotiq_85_left_knuckle_joint</param>
                     <param name="multiplier">-1</param>
-                    <xacro:unless value="${sim_ignition}">
+                    <xacro:unless value="${sim_ignition or sim_mujoco}">
                         <command_interface name="position"/>
                         <state_interface name="position"/>
@@ -79,5 +83,5 @@
                     <param name="mimic">${prefix}robotiq_85_left_knuckle_joint</param>
                     <param name="multiplier">-1</param>
-                    <xacro:unless value="${sim_ignition}">
+                    <xacro:unless value="${sim_ignition or sim_mujoco}">
                         <command_interface name="position"/>
                         <state_interface name="position"/>
@@ -88,5 +92,5 @@
                     <param name="mimic">${prefix}robotiq_85_left_knuckle_joint</param>
                     <param name="multiplier">1</param>
-                    <xacro:unless value="${sim_ignition}">
+                    <xacro:unless value="${sim_ignition or sim_mujoco}">
                         <command_interface name="position"/>
                         <state_interface name="position"/>
@@ -96,5 +100,5 @@
             </xacro:if>
             <!-- Only add this with fake hardware mode -->
-            <xacro:unless value="${sim_ignition or sim_isaac}">
+            <xacro:unless value="${sim_ignition or sim_isaac or sim_mujoco}">
                 <gpio name="reactivate_gripper">
                     <command_interface name="reactivate_gripper_cmd" />

File: ros2_ws/src/ros2_robotiq_gripper/robotiq_description/urdf/robotiq_2f_85_macro.urdf.xacro (robot description, xacro)
@@ -6,4 +6,5 @@
         parent
         *origin
+        sim_mujoco:=false
         sim_ignition:=false
         sim_isaac:=false
@@ -20,4 +21,5 @@
             <xacro:robotiq_gripper_ros2_control
                 name="${name}" prefix="${prefix}"
+                sim_mujoco="${sim_mujoco}"
                 sim_ignition="${sim_ignition}"
                 sim_isaac="${sim_isaac}"

File: ros2_ws/src/two_arm_moveit2_config/urdf/gen3_dual_arm.xacro (robot description, xacro)
@@ -5,5 +5,5 @@
     <xacro:arg name="dof" default="7" />
     <xacro:arg name="vision" default="false" />
-    <xacro:arg name="robot_ip" default="" />
+    <xacro:arg name="robot_ip" default="yyy.yyy.yyy.yyy" />
     <xacro:arg name="username" default="admin" />
     <xacro:arg name="password" default="admin" />
@@ -12,8 +12,9 @@
     <xacro:arg name="session_inactivity_timeout_ms" default="60000" />
     <xacro:arg name="connection_inactivity_timeout_ms" default="2000" />
-    <xacro:arg name="gripper" default="" />
+    <xacro:arg name="gripper" default="robotiq_2f_85" />
     <xacro:arg name="gripper_joint_name" default="" />
     <xacro:arg name="gripper_max_velocity" default="100.0" />
     <xacro:arg name="gripper_max_force" default="100.0" />
+    <xacro:arg name="sim_mujoco" default="false" />
     <xacro:arg name="sim_gazebo" default="false" />
     <xacro:arg name="sim_ignition" default="false" />
@@ -33,5 +34,7 @@
     </material>
     <!-- Initial positions from the YAML file -->
-    <xacro:property name="initial_positions_file" default="$(find two_arm_moveit2_config)/config/initial_positions.yaml"/>
+    <xacro:arg name="initial_positions_file" default="$(find two_arm_moveit2_config)/config/initial_positions.yaml"/>
+     <!-- convert to property to use substitution in function -->
+    <xacro:property name="initial_positions_file" default="$(arg initial_positions_file)"/>
     <!-- World link -->
     <link name="world">
@@ -78,5 +81,5 @@
     <origin rpy="0 0 0" xyz="-1.1125 0.80448 -0.09654"/>
     </joint>
-    <!-- Bin link -->
+    <!-- Bin link
     <link name="bin_link">
     <visual>
@@ -115,10 +118,10 @@
     </inertial>
     </link>
-    <!-- Bin joint -->
+    Bin joint
     <joint name="bin_joint" type="fixed">
     <parent link="world"/>
     <child link="bin_link"/>
     <origin xyz="0 0 0" rpy="0 0 0"/>
-    </joint>
+    </joint> -->
     <!-- Left arm -->
     <xacro:load_robot
@@ -142,4 +145,5 @@
         use_fake_hardware="$(arg use_fake_hardware)"
         fake_sensor_commands="$(arg fake_sensor_commands)"
+        sim_mujoco="$(arg sim_mujoco)"
         sim_gazebo="$(arg sim_gazebo)"
         sim_ignition="$(arg sim_ignition)"
@@ -170,4 +174,5 @@
         use_fake_hardware="$(arg use_fake_hardware)"
         fake_sensor_commands="$(arg fake_sensor_commands)"
+        sim_mujoco="$(arg sim_mujoco)"
         sim_gazebo="$(arg sim_gazebo)"
         sim_ignition="$(arg sim_ignition)"
