Commit message: fix gripper

File: ros2_ws/src/ros2_kortex/kortex_description/arms/gen3/7dof/urdf/kortex.ros2_control.xacro (robot description, xacro)
@@ -138,5 +138,5 @@
       <xacro:unless value="${use_fake_hardware or sim_gazebo or sim_ignition or sim_isaac}">
         <xacro:if value="${use_internal_bus_gripper_comm}">
-          <joint name="${prefix}${gripper_joint_name}">
+          <joint name="${gripper_joint_name}">
             <command_interface name="position" />
             <state_interface name="position"/>

File: ros2_ws/src/two_arm_moveit2_config/urdf/gen3_dual_arm.xacro (robot description, xacro)
@@ -382,5 +382,5 @@
         arm="$(arg arm)"
         gripper="$(arg gripper)"
-        gripper_joint_name="robotiq_85_left_knuckle_joint"
+        gripper_joint_name="left_robotiq_85_left_knuckle_joint"
         gripper_max_velocity="$(arg gripper_max_velocity)"
         gripper_max_force="$(arg gripper_max_force)"
@@ -410,5 +410,5 @@
         arm="$(arg arm)"
         gripper="$(arg gripper)"
-        gripper_joint_name="robotiq_85_left_knuckle_joint"
+        gripper_joint_name="right_robotiq_85_left_knuckle_joint"
         gripper_max_velocity="$(arg gripper_max_velocity)"
         gripper_max_force="$(arg gripper_max_force)"
