Commit message: yay

File: ros2_ws/src/two_arm_moveit2_config/urdf/gen3_dual_arm.urdf.xacro (robot description, xacro)
@@ -5,5 +5,5 @@
     <!-- Arguments -->
     <xacro:arg name="prefix" default="" />
-    <xacro:arg name="arm" default="NO_ARM_TYPE_DEFINED" />
+    <xacro:arg name="arm" default="gen3" />
     <xacro:arg name="dof" default="7" />
     <xacro:arg name="vision" default="false" />
@@ -64,5 +64,5 @@
         <origin rpy="1.5708 0 0" xyz="0 0 0"/>
         <geometry>
-        <mesh filename="package://control/kinova_gen3_mujoco/assets/VentionAssembly.stl" scale="0.001 0.001 0.001"/>
+        <mesh filename="file://$(find control)/kinova_gen3_mujoco/assets/VentionAssembly.stl" scale="0.001 0.001 0.001"/>
         </geometry>
         <material name="dark_blue_metal"/>
@@ -71,5 +71,5 @@
         <origin rpy="1.5708 0 0" xyz="0 0 0"/>
         <geometry>
-        <mesh filename="package://control/kinova_gen3_mujoco/assets/VentionAssembly.stl" scale="0.001 0.001 0.001"/>
+        <mesh filename="file://$(find control)/kinova_gen3_mujoco/assets/VentionAssembly.stl" scale="0.001 0.001 0.001"/>
         </geometry>
     </collision>
@@ -90,5 +90,5 @@
     <visual>
         <geometry>
-        <mesh filename="package://control/kinova_gen3_mujoco/assets/bin.stl" scale="0.001 0.001 0.001"/>
+        <mesh filename="file://$(find control)/kinova_gen3_mujoco/assets/bin.stl" scale="0.001 0.001 0.001"/>
         </geometry>
         <material name="bin_material"/>
@@ -97,5 +97,5 @@
     <collision>
         <geometry>
-        <mesh filename="package://control/kinova_gen3_mujoco/assets/bin.stl" scale="0.001 0.001 0.001"/>
+        <mesh filename="file://$(find control)/kinova_gen3_mujoco/assets/bin.stl" scale="0.001 0.001 0.001"/>
         </geometry>
         <origin xyz="-0.1905 0.15875 0.9316" rpy="1.5708 0 0"/>

Commit message: some changes

File: ros2_ws/src/two_arm_moveit2_config/urdf/gen3_dual_arm.urdf.xacro (robot description, xacro)
@@ -135,5 +135,5 @@
         arm="$(arg arm)"
         gripper="$(arg gripper)"
-        gripper_joint_name="left_robotiq_85_left_knuckle_joint"
+        gripper_joint_name="robotiq_85_left_knuckle_joint"
         gripper_max_velocity="$(arg gripper_max_velocity)"
         gripper_max_force="$(arg gripper_max_force)"
@@ -163,5 +163,5 @@
         arm="$(arg arm)"
         gripper="$(arg gripper)"
-        gripper_joint_name="right_robotiq_85_left_knuckle_joint"
+        gripper_joint_name="robotiq_85_left_knuckle_joint"
         gripper_max_velocity="$(arg gripper_max_velocity)"
         gripper_max_force="$(arg gripper_max_force)"

File: ros2_ws/src/two_arm_moveit2_config/urdf/gen3_dual_arm.xacro (robot description, xacro)
@@ -81,5 +81,5 @@
     <origin rpy="0 0 0" xyz="-1.1125 0.80448 -0.09654"/>
     </joint>
-    <!-- Bin link -->
+    <!-- Bin link
     <link name="bin_link">
     <visual>
@@ -118,10 +118,10 @@
     </inertial>
     </link>
-    <!-- Bin joint -->
+    Bin joint
     <joint name="bin_joint" type="fixed">
     <parent link="world"/>
     <child link="bin_link"/>
     <origin xyz="0 0 0" rpy="0 0 0"/>
-    </joint>
+    </joint> -->
     <link name="bound_top_link">
     <visual>
@@ -386,5 +386,5 @@
         arm="$(arg arm)"
         gripper="$(arg gripper)"
-        gripper_joint_name="left_robotiq_85_left_knuckle_joint"
+        gripper_joint_name="robotiq_85_left_knuckle_joint"
         gripper_max_velocity="$(arg gripper_max_velocity)"
         gripper_max_force="$(arg gripper_max_force)"
@@ -414,5 +414,5 @@
         arm="$(arg arm)"
         gripper="$(arg gripper)"
-        gripper_joint_name="right_robotiq_85_left_knuckle_joint"
+        gripper_joint_name="robotiq_85_left_knuckle_joint"
         gripper_max_velocity="$(arg gripper_max_velocity)"
         gripper_max_force="$(arg gripper_max_force)"

Commit message: get bin

File: ros2_ws/src/two_arm_moveit2_config/urdf/gen3_dual_arm.urdf.xacro (robot description, xacro)
@@ -86,5 +86,5 @@
     <origin rpy="0 0 0" xyz="-1.1125 0.80448 -0.09654"/>
     </joint>
-    <!-- Bin link -->
+    <!-- Bin link
     <link name="bin_link">
     <visual>
@@ -123,10 +123,9 @@
     </inertial>
     </link>
-    <!-- Bin joint -->
     <joint name="bin_joint" type="fixed">
     <parent link="world"/>
     <child link="bin_link"/>
     <origin xyz="0 0 0" rpy="0 0 0"/>
-    </joint>
+    </joint> -->
     <!-- Left arm -->
     <xacro:load_robot

File: ros2_ws/src/two_arm_moveit2_config/urdf/gen3_dual_arm.xacro (robot description, xacro)
@@ -81,11 +81,6 @@
     <origin rpy="0 0 0" xyz="-1.1125 0.80448 -0.09654"/>
     </joint>
-<<<<<<< HEAD
     <!-- Bin link
     <link name="bin_link">
-=======
-    <!-- Bin link -->
-    <!-- <link name="bin_link">
->>>>>>> mlee/fsm
     <visual>
         <geometry>

Commit message: bin in sim

File: ros2_ws/src/two_arm_moveit2_config/urdf/gen3_dual_arm.urdf.xacro (robot description, xacro)
@@ -85,47 +85,4 @@
     <child link="vention_table_link"/>
     <origin rpy="0 0 0" xyz="-1.1125 0.80448 -0.09654"/>
-    </joint>
-    <!-- Bin link -->
-    <link name="bin_link">
-    <visual>
-        <geometry>
-        <mesh filename="file://$(find control)/kinova_gen3_mujoco/assets/bin.stl" scale="0.001 0.001 0.001"/>
-        </geometry>
-        <material name="bin_material"/>
-        <origin xyz="-0.1905 0.15875 0.9316" rpy="1.5708 0 0"/>
-    </visual>
-    <collision>
-        <geometry>
-        <mesh filename="file://$(find control)/kinova_gen3_mujoco/assets/bin.stl" scale="0.001 0.001 0.001"/>
-        </geometry>
-        <origin xyz="-0.1905 0.15875 0.9316" rpy="1.5708 0 0"/>
-        <surface>
-        <friction>
-            <ode>
-            <mu1>1.0</mu1>
-            <mu2>1.0</mu2>
-            </ode>
-        </friction>
-        <contact>
-            <ode>
-            <kp>1000.0</kp>
-            <kd>100.0</kd>
-            <max_vel>0.01</max_vel>
-            <min_depth>0.001</min_depth>
-            </ode>
-        </contact>
-        </surface>
-    </collision>
-    <inertial>
-        <mass value="0.68"/>
-        <origin xyz="-0.1905 0.15875 0.9316" rpy="1.5708 0 0"/>
-        <inertia ixx="0.001" ixy="0.0" ixz="0.0" iyy="0.001" iyz="0.0" izz="0.001"/>
-    </inertial>
-    </link>
-    <!-- Bin joint -->
-    <joint name="bin_joint" type="fixed">
-    <parent link="world"/>
-    <child link="bin_link"/>
-    <origin xyz="0 0 0" rpy="0 0 0"/>
     </joint>
     <!-- Left arm -->
