Commit message: get rid of junk

File: ros2_ws/src/two_arm_moveit2_config/urdf/gen3_dual_arm.xacro (robot description, xacro)
@@ -127,50 +127,4 @@
     <origin xyz="0 0 0" rpy="0 0 0"/>
     </joint>
-    <!-- <xacro:load_robot
-        parent="world"
-        arm="gen3"
-        gripper="$(arg gripper)"
-        dof="7"
-        vision="$(arg vision)"
-        prefix="$(arg left_prefix)"
-        gripper_joint_name="finger_joint"
-        robot_ip="192.168.1.10"
-        username="admin"
-        password="admin"
-        port="10000"
-        port_realtime="10001"
-        session_inactivity_timeout_ms="60000"
-        connection_inactivity_timeout_ms="2000"
-        use_fake_hardware="true"
-        fake_sensor_commands="false"
-        sim_gazebo="false"
-        sim_ignition="false"
-        sim_isaac="false"
-        initial_positions="${xacro.load_yaml(initial_positions_file)}" >
-        <origin rpy="0 0 3.14" xyz="0.63017298 0 0.93657"/>
-    </xacro:load_robot>
-    <xacro:load_robot
-        parent="world"
-        arm="gen3"
-        gripper="$(arg gripper)"
-        dof="7"
-        vision="$(arg vision)"
-        prefix="$(arg right_prefix)"
-        gripper_joint_name="finger_joint"
-        robot_ip="192.168.1.11"
-        username="admin"
-        password="admin"
-        port="10000"
-        port_realtime="10001"
-        session_inactivity_timeout_ms="60000"
-        connection_inactivity_timeout_ms="2000"
-        use_fake_hardware="true"
-        fake_sensor_commands="false"
-        sim_gazebo="false"
-        sim_ignition="false"
-        sim_isaac="false"
-        initial_positions="${xacro.load_yaml(initial_positions_file)}" >
-        <origin rpy="0 0 0" xyz="-0.63017298 0 0.93657"/>
-    </xacro:load_robot> -->
     <!-- Left arm -->
     <xacro:load_robot
@@ -229,25 +183,3 @@
         <origin rpy="0 0 0" xyz="-0.63017298 0 0.93657"/>
     </xacro:load_robot>
-    <!-- Left gripper
-    <xacro:load_gripper
-        parent="left_end_effector_link"
-        prefix="left_"
-        use_fake_hardware="false"
-        fake_sensor_commands="false"
-        sim_ignition="false"
-        sim_isaac="false"
-        com_port="/dev/ttyUSB0"
-        use_internal_bus_gripper_comm="false"
-        moveit_active="false"/>
-    Right gripper
-    <xacro:load_gripper
-        parent="right_end_effector_link"
-        prefix="right_"
-        use_fake_hardware="false"
-        fake_sensor_commands="false"
-        sim_ignition="false"
-        sim_isaac="false"
-        com_port="/dev/ttyUSB0"
-        use_internal_bus_gripper_comm="false"
-        moveit_active="false"/> -->
 </robot>

Commit message: get gripper working

File: ros2_ws/src/two_arm_moveit2_config/urdf/gen3_dual_arm.xacro (robot description, xacro)
@@ -5,5 +5,5 @@
     <xacro:arg name="dof" default="7" />
     <xacro:arg name="vision" default="false" />
-    <xacro:arg name="robot_ip" default="192.168.11.11" />
+    <xacro:arg name="robot_ip" default="" />
     <xacro:arg name="username" default="admin" />
     <xacro:arg name="password" default="admin" />
@@ -132,5 +132,5 @@
         dof="$(arg dof)"
         vision="$(arg vision)"
-        robot_ip="192.168.1.10"
+        robot_ip="192.168.1.41"
         username="admin"
         password="admin"
@@ -139,5 +139,5 @@
         session_inactivity_timeout_ms="60000"
         connection_inactivity_timeout_ms="60000"
-        use_internal_bus_gripper_comm="false"
+        use_internal_bus_gripper_comm="true"
         use_fake_hardware="$(arg use_fake_hardware)"
         fake_sensor_commands="$(arg fake_sensor_commands)"
@@ -147,5 +147,5 @@
         use_external_cable="$(arg use_external_cable)"
         initial_positions="${xacro.load_yaml(initial_positions_file)}" >
-        <origin rpy="0 0 3.14" xyz="0.63017298 0 0.93657"/>  position robot in the world
+        <origin rpy="0 0 3.14" xyz="0.63017298 0 0.93657"/>
     </xacro:load_robot>
     <!-- Right arm -->
@@ -160,5 +160,5 @@
         dof="$(arg dof)"
         vision="$(arg vision)"
-        robot_ip="192.168.1.10"
+        robot_ip="192.168.1.42"
         username="admin"
         password="admin"
@@ -167,5 +167,5 @@
         session_inactivity_timeout_ms="60000"
         connection_inactivity_timeout_ms="60000"
-        use_internal_bus_gripper_comm="false"
+        use_internal_bus_gripper_comm="true"
         use_fake_hardware="$(arg use_fake_hardware)"
         fake_sensor_commands="$(arg fake_sensor_commands)"

Commit message: gripper with collision aware and extra padding
Added gripper into planning group
Included home pose
Added padding
Resolved padding's collision conflicts with table

File: ros2_ws/src/two_arm_moveit2_config/urdf/gen3_dual_arm.xacro (robot description, xacro)
@@ -120,4 +120,260 @@
     <child link="bin_link"/>
     <origin xyz="0 0 0" rpy="0 0 0"/>
+    </joint>
+    <link name="bound_top_link">
+    <visual>
+        <geometry>
+        <box size="1.5 0.1 0.1"/>
+        </geometry>
+        <material name="dark_blue_metal"/>
+    </visual>
+    <collision>
+        <geometry>
+        <box size="1.5 0.1 0.1"/>
+        </geometry>
+    </collision>
+    <inertial>
+        <mass value="1.0"/>
+        <inertia
+        ixx="0.00167"
+        ixy="0.0"
+        ixz="0.0"
+        iyy="0.33417"
+        iyz="0.0"
+        izz="0.33417"/>
+    </inertial>
+    </link>
+    <joint name="bound_top_joint" type="fixed">
+    <parent link="world"/>
+    <child link="bound_top_link"/>
+    <origin rpy="0 0 0" xyz="0 0 1.8"/>
+    </joint>
+    <link name="bound_left_link">
+    <visual>
+        <geometry>
+        <box size="1 0.1 0.1"/>
+        </geometry>
+        <material name="dark_blue_metal"/>
+    </visual>
+    <collision>
+        <geometry>
+        <box size="1 0.1 0.1"/>
+        </geometry>
+    </collision>
+    <inertial>
+        <mass value="1.0"/>
+        <inertia
+        ixx="0.00167"
+        ixy="0.0"
+        ixz="0.0"
+        iyy="0.33417"
+        iyz="0.0"
+        izz="0.33417"/>
+    </inertial>
+    </link>
+    <joint name="bound_left_joint" type="fixed">
+    <parent link="world"/>
+    <child link="bound_left_link"/>
+    <origin rpy="0 0 1.5708" xyz="0.75 0 1.8"/>
+    </joint>
+    <!-- Simple box link -->
+    <link name="bound_right_link">
+    <visual>
+        <geometry>
+        <box size="1 0.1 0.1"/>
+        </geometry>
+        <material name="dark_blue_metal"/>
+    </visual>
+    <collision>
+        <geometry>
+        <box size="1 0.1 0.1"/>
+        </geometry>
+    </collision>
+    <inertial>
+        <mass value="1.0"/>
+        <inertia
+        ixx="0.00167"
+        ixy="0.0"
+        ixz="0.0"
+        iyy="0.33417"
+        iyz="0.0"
+        izz="0.33417"/>
+    </inertial>
+    </link>
+    <joint name="bound_right_joint" type="fixed">
+    <parent link="world"/>
+    <child link="bound_right_link"/>
+    <origin rpy="0 0 1.5708" xyz="-0.7 0 1.8"/>
+    </joint>
+    <link name="bound_right_top_link">
+    <visual>
+        <geometry>
+        <box size="1 0.1 0.1"/>
+        </geometry>
+        <material name="dark_blue_metal"/>
+    </visual>
+    <collision>
+        <geometry>
+        <box size="1 0.1 0.1"/>
+        </geometry>
+    </collision>
+    <inertial>
+        <mass value="1.0"/>
+        <inertia
+        ixx="0.00167"
+        ixy="0.0"
+        ixz="0.0"
+        iyy="0.33417"
+        iyz="0.0"
+        izz="0.33417"/>
+    </inertial>
+    </link>
+    <joint name="bound_right_top_joint" type="fixed">
+    <parent link="world"/>
+    <child link="bound_right_top_link"/>
+    <origin rpy="0 0 1.5708" xyz="-0.7 0 2.03"/>
+    </joint>
+    <!-- Simple box link -->
+    <link name="bound_left_top_link">
+    <visual>
+        <geometry>
+        <box size="1 0.1 0.1"/>
+        </geometry>
+        <material name="dark_blue_metal"/>
+    </visual>
+    <collision>
+        <geometry>
+        <box size="1 0.1 0.1"/>
+        </geometry>
+    </collision>
+    <inertial>
+        <mass value="1.0"/>
+        <inertia
+        ixx="0.00167"
+        ixy="0.0"
+        ixz="0.0"
+        iyy="0.33417"
+        iyz="0.0"
+        izz="0.33417"/>
+    </inertial>
+    </link>
+    <joint name="bound_left_top_joint" type="fixed">
+    <parent link="world"/>
+    <child link="bound_left_top_link"/>
+    <origin rpy="0 0 1.5708" xyz="0.75 0 2.03"/>
+    </joint>
+    <!-- Simple box link -->
+    <link name="bound_stand_1_link">
+    <visual>
+        <geometry>
+        <box size="2 0.1 0.1"/>
+        </geometry>
+        <material name="dark_blue_metal"/>
+    </visual>
+    <collision>
+        <geometry>
+        <box size="2 0.1 0.1"/>
+        </geometry>
+    </collision>
+    <inertial>
+        <mass value="1.0"/>
+        <inertia
+        ixx="0.00167"
+        ixy="0.0"
+        ixz="0.0"
+        iyy="0.33417"
+        iyz="0.0"
+        izz="0.33417"/>
+    </inertial>
+    </link>
+    <joint name="bound_stand_1_joint" type="fixed">
+    <parent link="world"/>
+    <child link="bound_stand_1_link"/>
+    <origin rpy="0 1.5708 0" xyz="0.75 -0.55 1.1"/>
+    </joint>
+    <!-- Simple box link -->
+    <link name="bound_stand_2_link">
+    <visual>
+        <geometry>
+        <box size="2 0.1 0.1"/>
+        </geometry>
+        <material name="dark_blue_metal"/>
+    </visual>
+    <collision>
+        <geometry>
+        <box size="2 0.1 0.1"/>
+        </geometry>
+    </collision>
+    <inertial>
+        <mass value="1.0"/>
+        <inertia
+        ixx="0.00167"
+        ixy="0.0"
+        ixz="0.0"
+        iyy="0.33417"
+        iyz="0.0"
+        izz="0.33417"/>
+    </inertial>
+    </link>
+    <joint name="bound_stand_2_joint" type="fixed">
+    <parent link="world"/>
+    <child link="bound_stand_2_link"/>
+    <origin rpy="0 1.5708 0" xyz="-0.7 -0.55 1.1"/>
+    </joint>
+    <link name="bound_stand_3_link">
+    <visual>
+        <geometry>
+        <box size="2 0.1 0.1"/>
+        </geometry>
+        <material name="dark_blue_metal"/>
+    </visual>
+    <collision>
+        <geometry>
+        <box size="2 0.1 0.1"/>
+        </geometry>
+    </collision>
+    <inertial>
+        <mass value="1.0"/>
+        <inertia
+        ixx="0.00167"
+        ixy="0.0"
+        ixz="0.0"
+        iyy="0.33417"
+        iyz="0.0"
+        izz="0.33417"/>
+    </inertial>
+    </link>
+    <joint name="bound_stand_3_joint" type="fixed">
+    <parent link="world"/>
+    <child link="bound_stand_3_link"/>
+    <origin rpy="0 1.5708 0" xyz="-0.7 0.55 1.1"/>
+    </joint>
+    <link name="bound_stand_4_link">
+    <visual>
+        <geometry>
+        <box size="2 0.1 0.1"/>
+        </geometry>
+        <material name="dark_blue_metal"/>
+    </visual>
+    <collision>
+        <geometry>
+        <box size="2 0.1 0.1"/>
+        </geometry>
+    </collision>
+    <inertial>
+        <mass value="1.0"/>
+        <inertia
+        ixx="0.00167"
+        ixy="0.0"
+        ixz="0.0"
+        iyy="0.33417"
+        iyz="0.0"
+        izz="0.33417"/>
+    </inertial>
+    </link>
+    <joint name="bound_stand_4_joint" type="fixed">
+    <parent link="world"/>
+    <child link="bound_stand_4_link"/>
+    <origin rpy="0 1.5708 0" xyz="0.75 0.55 1.1"/>
     </joint>
     <!-- Left arm -->

Commit message: Mlee/ros node traj (#14)

File: ros2_ws/src/two_arm_moveit2_config/urdf/gen3_dual_arm.xacro (robot description, xacro)
@@ -5,5 +5,5 @@
     <xacro:arg name="dof" default="7" />
     <xacro:arg name="vision" default="false" />
-    <xacro:arg name="robot_ip" default="192.168.11.11" />
+    <xacro:arg name="robot_ip" default="" />
     <xacro:arg name="username" default="admin" />
     <xacro:arg name="password" default="admin" />
@@ -388,5 +388,5 @@
         dof="$(arg dof)"
         vision="$(arg vision)"
-        robot_ip="192.168.1.10"
+        robot_ip="192.168.1.41"
         username="admin"
         password="admin"
@@ -395,5 +395,5 @@
         session_inactivity_timeout_ms="60000"
         connection_inactivity_timeout_ms="60000"
-        use_internal_bus_gripper_comm="false"
+        use_internal_bus_gripper_comm="true"
         use_fake_hardware="$(arg use_fake_hardware)"
         fake_sensor_commands="$(arg fake_sensor_commands)"
@@ -403,5 +403,5 @@
         use_external_cable="$(arg use_external_cable)"
         initial_positions="${xacro.load_yaml(initial_positions_file)}" >
-        <origin rpy="0 0 3.14" xyz="0.63017298 0 0.93657"/>  position robot in the world
+        <origin rpy="0 0 3.14" xyz="0.63017298 0 0.93657"/>
     </xacro:load_robot>
     <!-- Right arm -->
@@ -416,5 +416,5 @@
         dof="$(arg dof)"
         vision="$(arg vision)"
-        robot_ip="192.168.1.10"
+        robot_ip="192.168.1.42"
         username="admin"
         password="admin"
@@ -423,5 +423,5 @@
         session_inactivity_timeout_ms="60000"
         connection_inactivity_timeout_ms="60000"
-        use_internal_bus_gripper_comm="false"
+        use_internal_bus_gripper_comm="true"
         use_fake_hardware="$(arg use_fake_hardware)"
         fake_sensor_commands="$(arg fake_sensor_commands)"

Commit message: we're getting somewhere. where? who knows

File: ros2_ws/src/two_arm_moveit2_config/urdf/gen3_dual_arm.xacro (robot description, xacro)
@@ -52,5 +52,5 @@
     </link>
     <!-- Table link -->
-    <link name="vention_table_link">
+    <!-- <link name="vention_table_link">
     <visual>
         <origin rpy="1.5708 0 0" xyz="0 0 0"/>
@@ -72,5 +72,5 @@
     </inertial>
     </link>
-    <!-- Table joint -->
+    Table joint
     <joint name="table_joint" type="fixed">
     <parent link="world"/>
@@ -78,5 +78,5 @@
     <origin rpy="0 0 0" xyz="-1.1125 0.80448 -0.09654"/>
     </joint>
-    <!-- Bin link -->
+    Bin link
     <link name="bin_link">
     <visual>
@@ -115,5 +115,5 @@
     </inertial>
     </link>
-    <!-- Bin joint -->
+    Bin joint
     <joint name="bin_joint" type="fixed">
     <parent link="world"/>
@@ -121,4 +121,5 @@
     <origin xyz="0 0 0" rpy="0 0 0"/>
     </joint>
+    Collision boxes
     <link name="bound_top_link">
     <visual>
@@ -177,5 +178,4 @@
     <origin rpy="0 0 1.5708" xyz="0.75 0 1.8"/>
     </joint>
-    <!-- Simple box link -->
     <link name="bound_right_link">
     <visual>
@@ -234,5 +234,4 @@
     <origin rpy="0 0 1.5708" xyz="-0.7 0 2.03"/>
     </joint>
-    <!-- Simple box link -->
     <link name="bound_left_top_link">
     <visual>
@@ -263,5 +262,4 @@
     <origin rpy="0 0 1.5708" xyz="0.75 0 2.03"/>
     </joint>
-    <!-- Simple box link -->
     <link name="bound_stand_1_link">
     <visual>
@@ -292,5 +290,4 @@
     <origin rpy="0 1.5708 0" xyz="0.75 -0.55 1.1"/>
     </joint>
-    <!-- Simple box link -->
     <link name="bound_stand_2_link">
     <visual>
@@ -376,5 +373,5 @@
     <child link="bound_stand_4_link"/>
     <origin rpy="0 1.5708 0" xyz="0.75 0.55 1.1"/>
-    </joint>
+    </joint> -->
     <!-- Left arm -->
     <xacro:load_robot

Commit message: get rid of boxes

File: ros2_ws/src/two_arm_moveit2_config/urdf/gen3_dual_arm.xacro (robot description, xacro)
@@ -121,5 +121,5 @@
     <origin xyz="0 0 0" rpy="0 0 0"/>
     </joint>
-    <link name="bound_top_link">
+    <!-- <link name="bound_top_link">
     <visual>
         <geometry>
@@ -177,5 +177,4 @@
     <origin rpy="0 0 1.5708" xyz="0.75 0 1.8"/>
     </joint>
-    <!-- Simple box link -->
     <link name="bound_right_link">
     <visual>
@@ -234,5 +233,4 @@
     <origin rpy="0 0 1.5708" xyz="-0.7 0 2.03"/>
     </joint>
-    <!-- Simple box link -->
     <link name="bound_left_top_link">
     <visual>
@@ -263,5 +261,4 @@
     <origin rpy="0 0 1.5708" xyz="0.75 0 2.03"/>
     </joint>
-    <!-- Simple box link -->
     <link name="bound_stand_1_link">
     <visual>
@@ -292,5 +289,4 @@
     <origin rpy="0 1.5708 0" xyz="0.75 -0.55 1.1"/>
     </joint>
-    <!-- Simple box link -->
     <link name="bound_stand_2_link">
     <visual>
@@ -376,5 +372,5 @@
     <child link="bound_stand_4_link"/>
     <origin rpy="0 1.5708 0" xyz="0.75 0.55 1.1"/>
-    </joint>
+    </joint> -->
     <!-- Left arm -->
     <xacro:load_robot

Commit message: motion planning fsm

File: ros2_ws/src/two_arm_moveit2_config/urdf/gen3_dual_arm.xacro (robot description, xacro)
@@ -121,5 +121,5 @@
     <origin xyz="0 0 0" rpy="0 0 0"/>
     </joint>
-    <!-- <link name="bound_top_link">
+    <link name="bound_top_link">
     <visual>
         <geometry>
@@ -372,5 +372,5 @@
     <child link="bound_stand_4_link"/>
     <origin rpy="0 1.5708 0" xyz="0.75 0.55 1.1"/>
-    </joint> -->
+    </joint>
     <!-- Left arm -->
     <xacro:load_robot

Commit message: move to grasp

File: ros2_ws/src/two_arm_moveit2_config/urdf/gen3_dual_arm.xacro (robot description, xacro)
@@ -78,5 +78,5 @@
     <origin rpy="0 0 0" xyz="-1.1125 0.80448 -0.09654"/>
     </joint>
-    <!-- Bin link -->
+    <!-- Bin link
     <link name="bin_link">
     <visual>
@@ -115,5 +115,5 @@
     </inertial>
     </link>
-    <!-- Bin joint -->
+    Bin joint
     <joint name="bin_joint" type="fixed">
     <parent link="world"/>
@@ -143,5 +143,5 @@
         izz="0.33417"/>
     </inertial>
-    </link>
+    </link> -->
     <joint name="bound_top_joint" type="fixed">
     <parent link="world"/>

Commit message: reduced padding and made it transparent

File: ros2_ws/src/two_arm_moveit2_config/urdf/gen3_dual_arm.xacro (robot description, xacro)
@@ -29,4 +29,7 @@
     <color rgba="0.0 0.1 0.2 1"/>
     </material>
+    <material name="transparent">
+    <color rgba="0.8 0.8 0.8 0"/>
+    </material>
     <material name="bin_material">
     <color rgba="0.25 0.25 0.25 1"/>
@@ -124,11 +127,11 @@
     <visual>
         <geometry>
-        <box size="1.5 0.1 0.1"/>
-        </geometry>
-        <material name="dark_blue_metal"/>
-    </visual>
-    <collision>
-        <geometry>
-        <box size="1.5 0.1 0.1"/>
+        <box size="1.5 0.06 0.06"/>
+        </geometry>
+        <material name="transparent"/>
+    </visual>
+    <collision>
+        <geometry>
+        <box size="1.5 0.06 0.06"/>
         </geometry>
     </collision>
@@ -152,11 +155,11 @@
     <visual>
         <geometry>
-        <box size="1 0.1 0.1"/>
-        </geometry>
-        <material name="dark_blue_metal"/>
-    </visual>
-    <collision>
-        <geometry>
-        <box size="1 0.1 0.1"/>
+        <box size="1 0.06 0.06"/>
+        </geometry>
+        <material name="transparent"/>
+    </visual>
+    <collision>
+        <geometry>
+        <box size="1 0.06 0.06"/>
         </geometry>
     </collision>
@@ -181,11 +184,11 @@
     <visual>
         <geometry>
-        <box size="1 0.1 0.1"/>
-        </geometry>
-        <material name="dark_blue_metal"/>
-    </visual>
-    <collision>
-        <geometry>
-        <box size="1 0.1 0.1"/>
+        <box size="1 0.06 0.06"/>
+        </geometry>
+        <material name="transparent"/>
+    </visual>
+    <collision>
+        <geometry>
+        <box size="1 0.06 0.06"/>
         </geometry>
     </collision>
@@ -204,16 +207,16 @@
     <parent link="world"/>
     <child link="bound_right_link"/>
-    <origin rpy="0 0 1.5708" xyz="-0.7 0 1.8"/>
+    <origin rpy="0 0 1.5708" xyz="-0.73 0 1.8"/>
     </joint>
     <link name="bound_right_top_link">
     <visual>
         <geometry>
-        <box size="1 0.1 0.1"/>
-        </geometry>
-        <material name="dark_blue_metal"/>
-    </visual>
-    <collision>
-        <geometry>
-        <box size="1 0.1 0.1"/>
+        <box size="1 0.06 0.06"/>
+        </geometry>
+        <material name="transparent"/>
+    </visual>
+    <collision>
+        <geometry>
+        <box size="1 0.06 0.06"/>
         </geometry>
     </collision>
@@ -232,5 +235,5 @@
     <parent link="world"/>
     <child link="bound_right_top_link"/>
-    <origin rpy="0 0 1.5708" xyz="-0.7 0 2.03"/>
+    <origin rpy="0 0 1.5708" xyz="-0.73 0 2.03"/>
     </joint>
     <!-- Simple box link -->
@@ -238,17 +241,17 @@
     <visual>
         <geometry>
-        <box size="1 0.1 0.1"/>
-        </geometry>
-        <material name="dark_blue_metal"/>
-    </visual>
-    <collision>
-        <geometry>
-        <box size="1 0.1 0.1"/>
-        </geometry>
-    </collision>
-    <inertial>
-        <mass value="1.0"/>
-        <inertia
-        ixx="0.00167"
+        <box size="1 0.06 0.06"/>
+        </geometry>
+        <material name="transparent"/>
+    </visual>
+    <collision>
+        <geometry>
+        <box size="1 0.06 0.06"/>
+        </geometry>
+    </collision>
+    <inertial>
+        <mass value="1.0"/>
+        <inertia
+        ixx="0.0"
         ixy="0.0"
         ixz="0.0"
@@ -269,5 +272,5 @@
         <box size="2 0.1 0.1"/>
         </geometry>
-        <material name="dark_blue_metal"/>
+        <material name="transparent"/>
     </visual>
     <collision>
@@ -298,5 +301,5 @@
         <box size="2 0.1 0.1"/>
         </geometry>
-        <material name="dark_blue_metal"/>
+        <material name="transparent"/>
     </visual>
     <collision>
@@ -319,5 +322,5 @@
     <parent link="world"/>
     <child link="bound_stand_2_link"/>
-    <origin rpy="0 1.5708 0" xyz="-0.7 -0.55 1.1"/>
+    <origin rpy="0 1.5708 0" xyz="-0.73 -0.55 1.1"/>
     </joint>
     <link name="bound_stand_3_link">
@@ -326,5 +329,5 @@
         <box size="2 0.1 0.1"/>
         </geometry>
-        <material name="dark_blue_metal"/>
+        <material name="transparent"/>
     </visual>
     <collision>
@@ -347,5 +350,5 @@
     <parent link="world"/>
     <child link="bound_stand_3_link"/>
-    <origin rpy="0 1.5708 0" xyz="-0.7 0.55 1.1"/>
+    <origin rpy="0 1.5708 0" xyz="-0.73 0.55 1.1"/>
     </joint>
     <link name="bound_stand_4_link">
@@ -354,5 +357,5 @@
         <box size="2 0.1 0.1"/>
         </geometry>
-        <material name="dark_blue_metal"/>
+        <material name="transparent"/>
     </visual>
     <collision>

Commit message: progress

File: ros2_ws/src/two_arm_moveit2_config/urdf/gen3_dual_arm.xacro (robot description, xacro)
@@ -120,5 +120,5 @@
     <child link="bin_link"/>
     <origin xyz="0 0 0" rpy="0 0 0"/>
-    </joint>
+    </joint> -->
     <link name="bound_top_link">
     <visual>
@@ -143,5 +143,5 @@
         izz="0.33417"/>
     </inertial>
-    </link> -->
+    </link>
     <joint name="bound_top_joint" type="fixed">
     <parent link="world"/>

Commit message: add ros nodes

File: ros2_ws/src/two_arm_moveit2_config/urdf/gen3_dual_arm.xacro (robot description, xacro)
@@ -78,5 +78,5 @@
     <origin rpy="0 0 0" xyz="-1.1125 0.80448 -0.09654"/>
     </joint>
-    <!-- Bin link
+    <!-- Bin link -->
     <link name="bin_link">
     <visual>
@@ -115,10 +115,10 @@
     </inertial>
     </link>
-    Bin joint
+    <!-- Bin joint -->
     <joint name="bin_joint" type="fixed">
     <parent link="world"/>
     <child link="bin_link"/>
     <origin xyz="0 0 0" rpy="0 0 0"/>
-    </joint> -->
+    </joint>
     <link name="bound_top_link">
     <visual>
