Commit message: finish fsm for pick and place

File: ros2_ws/src/two_arm_moveit2_config/urdf/gen3_dual_arm.xacro (robot description, xacro)
@@ -79,5 +79,5 @@
     </joint>
     <!-- Bin link -->
-    <link name="bin_link">
+    <!-- <link name="bin_link">
     <visual>
         <geometry>
@@ -115,10 +115,10 @@
     </inertial>
     </link>
-    <!-- Bin joint -->
+    Bin joint
     <joint name="bin_joint" type="fixed">
     <parent link="world"/>
     <child link="bin_link"/>
     <origin xyz="0 0 0" rpy="0 0 0"/>
-    </joint>
+    </joint> -->
     <link name="bound_top_link">
     <visual>

Commit message: use IK to dual arm move

File: ros2_ws/src/two_arm_moveit2_config/urdf/gen3_dual_arm.xacro (robot description, xacro)
@@ -406,5 +406,5 @@
     <!-- Right arm -->
     <xacro:load_robot
-        parent="world"
+        parent="left_base_link"
         prefix="right_"
         arm="$(arg arm)"
@@ -430,5 +430,5 @@
         use_external_cable="$(arg use_external_cable)"
         initial_positions="${xacro.load_yaml(initial_positions_file)}" >
-        <origin rpy="0 0 0" xyz="-0.63017298 0 0.93657"/>
+        <origin rpy="0 0 -3.14" xyz="1.26034596 0 0"/>
     </xacro:load_robot>
 </robot>

Commit message: use cartesian, free up workspace, clean up code, lift and straight

File: ros2_ws/src/two_arm_moveit2_config/urdf/gen3_dual_arm.xacro (robot description, xacro)
@@ -28,10 +28,4 @@
     <material name="dark_blue_metal">
     <color rgba="0.0 0.1 0.2 1"/>
-    </material>
-    <material name="transparent">
-    <color rgba="0.8 0.8 0.8 0"/>
-    </material>
-    <material name="bin_material">
-    <color rgba="0.25 0.25 0.25 1"/>
     </material>
     <!-- Initial positions from the YAML file -->
@@ -80,299 +74,4 @@
     <child link="vention_table_link"/>
     <origin rpy="0 0 0" xyz="-1.1125 0.80448 -0.09654"/>
-    </joint>
-    <!-- Bin link
-    <link name="bin_link">
-    <visual>
-        <geometry>
-        <mesh filename="package://control/kinova_gen3_mujoco/assets/bin.stl" scale="0.001 0.001 0.001"/>
-        </geometry>
-        <material name="bin_material"/>
-        <origin xyz="-0.1905 0.15875 0.9316" rpy="1.5708 0 0"/>
-    </visual>
-    <collision>
-        <geometry>
-        <mesh filename="package://control/kinova_gen3_mujoco/assets/bin.stl" scale="0.001 0.001 0.001"/>
-        </geometry>
-        <origin xyz="-0.1905 0.15875 0.9316" rpy="1.5708 0 0"/>
-        <surface>
-        <friction>
-            <ode>
-            <mu1>1.0</mu1>
-            <mu2>1.0</mu2>
-            </ode>
-        </friction>
-        <contact>
-            <ode>
-            <kp>1000.0</kp>
-            <kd>100.0</kd>
-            <max_vel>0.01</max_vel>
-            <min_depth>0.001</min_depth>
-            </ode>
-        </contact>
-        </surface>
-    </collision>
-    <inertial>
-        <mass value="0.68"/>
-        <origin xyz="-0.1905 0.15875 0.9316" rpy="1.5708 0 0"/>
-        <inertia ixx="0.001" ixy="0.0" ixz="0.0" iyy="0.001" iyz="0.0" izz="0.001"/>
-    </inertial>
-    </link>
-    Bin joint
-    <joint name="bin_joint" type="fixed">
-    <parent link="world"/>
-    <child link="bin_link"/>
-    <origin xyz="0 0 0" rpy="0 0 0"/>
-    </joint> -->
-    <link name="bound_top_link">
-    <visual>
-        <geometry>
-        <box size="1.5 0.06 0.06"/>
-        </geometry>
-        <material name="transparent"/>
-    </visual>
-    <collision>
-        <geometry>
-        <box size="1.5 0.06 0.06"/>
-        </geometry>
-    </collision>
-    <inertial>
-        <mass value="1.0"/>
-        <inertia
-        ixx="0.00167"
-        ixy="0.0"
-        ixz="0.0"
-        iyy="0.33417"
-        iyz="0.0"
-        izz="0.33417"/>
-    </inertial>
-    </link>
-    <joint name="bound_top_joint" type="fixed">
-    <parent link="world"/>
-    <child link="bound_top_link"/>
-    <origin rpy="0 0 0" xyz="0 0 1.8"/>
-    </joint>
-    <link name="bound_left_link">
-    <visual>
-        <geometry>
-        <box size="1 0.06 0.06"/>
-        </geometry>
-        <material name="transparent"/>
-    </visual>
-    <collision>
-        <geometry>
-        <box size="1 0.06 0.06"/>
-        </geometry>
-    </collision>
-    <inertial>
-        <mass value="1.0"/>
-        <inertia
-        ixx="0.00167"
-        ixy="0.0"
-        ixz="0.0"
-        iyy="0.33417"
-        iyz="0.0"
-        izz="0.33417"/>
-    </inertial>
-    </link>
-    <joint name="bound_left_joint" type="fixed">
-    <parent link="world"/>
-    <child link="bound_left_link"/>
-    <origin rpy="0 0 1.5708" xyz="0.75 0 1.8"/>
-    </joint>
-    <link name="bound_right_link">
-    <visual>
-        <geometry>
-        <box size="1 0.06 0.06"/>
-        </geometry>
-        <material name="transparent"/>
-    </visual>
-    <collision>
-        <geometry>
-        <box size="1 0.06 0.06"/>
-        </geometry>
-    </collision>
-    <inertial>
-        <mass value="1.0"/>
-        <inertia
-        ixx="0.00167"
-        ixy="0.0"
-        ixz="0.0"
-        iyy="0.33417"
-        iyz="0.0"
-        izz="0.33417"/>
-    </inertial>
-    </link>
-    <joint name="bound_right_joint" type="fixed">
-    <parent link="world"/>
-    <child link="bound_right_link"/>
-    <origin rpy="0 0 1.5708" xyz="-0.73 0 1.8"/>
-    </joint>
-    <link name="bound_right_top_link">
-    <visual>
-        <geometry>
-        <box size="1 0.06 0.06"/>
-        </geometry>
-        <material name="transparent"/>
-    </visual>
-    <collision>
-        <geometry>
-        <box size="1 0.06 0.06"/>
-        </geometry>
-    </collision>
-    <inertial>
-        <mass value="1.0"/>
-        <inertia
-        ixx="0.00167"
-        ixy="0.0"
-        ixz="0.0"
-        iyy="0.33417"
-        iyz="0.0"
-        izz="0.33417"/>
-    </inertial>
-    </link>
-    <joint name="bound_right_top_joint" type="fixed">
-    <parent link="world"/>
-    <child link="bound_right_top_link"/>
-    <origin rpy="0 0 1.5708" xyz="-0.73 0 2.03"/>
-    </joint>
-    <link name="bound_left_top_link">
-    <visual>
-        <geometry>
-        <box size="1 0.06 0.06"/>
-        </geometry>
-        <material name="transparent"/>
-    </visual>
-    <collision>
-        <geometry>
-        <box size="1 0.06 0.06"/>
-        </geometry>
-    </collision>
-    <inertial>
-        <mass value="1.0"/>
-        <inertia
-        ixx="0.0"
-        ixy="0.0"
-        ixz="0.0"
-        iyy="0.33417"
-        iyz="0.0"
-        izz="0.33417"/>
-    </inertial>
-    </link>
-    <joint name="bound_left_top_joint" type="fixed">
-    <parent link="world"/>
-    <child link="bound_left_top_link"/>
-    <origin rpy="0 0 1.5708" xyz="0.75 0 2.03"/>
-    </joint>
-    <link name="bound_stand_1_link">
-    <visual>
-        <geometry>
-        <box size="2 0.1 0.1"/>
-        </geometry>
-        <material name="transparent"/>
-    </visual>
-    <collision>
-        <geometry>
-        <box size="2 0.1 0.1"/>
-        </geometry>
-    </collision>
-    <inertial>
-        <mass value="1.0"/>
-        <inertia
-        ixx="0.00167"
-        ixy="0.0"
-        ixz="0.0"
-        iyy="0.33417"
-        iyz="0.0"
-        izz="0.33417"/>
-    </inertial>
-    </link>
-    <joint name="bound_stand_1_joint" type="fixed">
-    <parent link="world"/>
-    <child link="bound_stand_1_link"/>
-    <origin rpy="0 1.5708 0" xyz="0.75 -0.55 1.1"/>
-    </joint>
-    <link name="bound_stand_2_link">
-    <visual>
-        <geometry>
-        <box size="2 0.1 0.1"/>
-        </geometry>
-        <material name="transparent"/>
-    </visual>
-    <collision>
-        <geometry>
-        <box size="2 0.1 0.1"/>
-        </geometry>
-    </collision>
-    <inertial>
-        <mass value="1.0"/>
-        <inertia
-        ixx="0.00167"
-        ixy="0.0"
-        ixz="0.0"
-        iyy="0.33417"
-        iyz="0.0"
-        izz="0.33417"/>
-    </inertial>
-    </link>
-    <joint name="bound_stand_2_joint" type="fixed">
-    <parent link="world"/>
-    <child link="bound_stand_2_link"/>
-    <origin rpy="0 1.5708 0" xyz="-0.73 -0.55 1.1"/>
-    </joint>
-    <link name="bound_stand_3_link">
-    <visual>
-        <geometry>
-        <box size="2 0.1 0.1"/>
-        </geometry>
-        <material name="transparent"/>
-    </visual>
-    <collision>
-        <geometry>
-        <box size="2 0.1 0.1"/>
-        </geometry>
-    </collision>
-    <inertial>
-        <mass value="1.0"/>
-        <inertia
-        ixx="0.00167"
-        ixy="0.0"
-        ixz="0.0"
-        iyy="0.33417"
-        iyz="0.0"
-        izz="0.33417"/>
-    </inertial>
-    </link>
-    <joint name="bound_stand_3_joint" type="fixed">
-    <parent link="world"/>
-    <child link="bound_stand_3_link"/>
-    <origin rpy="0 1.5708 0" xyz="-0.73 0.55 1.1"/>
-    </joint>
-    <link name="bound_stand_4_link">
-    <visual>
-        <geometry>
-        <box size="2 0.1 0.1"/>
-        </geometry>
-        <material name="transparent"/>
-    </visual>
-    <collision>
-        <geometry>
-        <box size="2 0.1 0.1"/>
-        </geometry>
-    </collision>
-    <inertial>
-        <mass value="1.0"/>
-        <inertia
-        ixx="0.00167"
-        ixy="0.0"
-        ixz="0.0"
-        iyy="0.33417"
-        iyz="0.0"
-        izz="0.33417"/>
-    </inertial>
-    </link>
-    <joint name="bound_stand_4_joint" type="fixed">
-    <parent link="world"/>
-    <child link="bound_stand_4_link"/>
-    <origin rpy="0 1.5708 0" xyz="0.75 0.55 1.1"/>
     </joint>
     <!-- Left arm -->
